Commit message: Uploading and updating URDF and USD files

File: isaac_sim/Main_Robot_L_URDF_tool.urdf (robot description, URDF)
Before this commit: robot Main_Robot_L_URDF, 7 links, 6 joints
Links:
- removed link forearm
- removed link link1
- removed link tcp
- removed link upper_arm
- removed link wrist
- added link link_1, mass 340; collision box size=0.42 0.38 0.32; collision cylinder length=0.36 radius=0.24
- added link link_2, mass 280; collision box size=1.30 0.26 0.24; visual box size=0.70 0.04 0.18
- added link link_3, mass 260; collision box size=1.35 0.20 0.18; visual box size=1.20 0.08 0.04
- added link link_4, mass 80; collision cylinder length=0.20 radius=0.12; visual cylinder length=0.08 radius=0.10
- link tool: geometry collision cylinder length=0.089084 radius=0.075; visual cylinder length=0.02 radius=0.04
Joints:
- removed joint A5
- removed joint joint1
- removed joint joint2
- removed joint joint3
- removed joint joint4
- removed joint tcp_fixed
- added joint joint_1: type revolute, parent base_link, child link_1, origin xyz=0 0 0.53, axis 0 0 1, limit lower=-3.22886 upper=3.22886 effort=50000 velocity=2.0
- added joint joint_2: type revolute, parent link_1, child link_2, origin xyz=0.350 0 0, axis 0 1 0, limit lower=-3.28122 upper=0.61087 effort=25000 velocity=2.0
- added joint joint_3: type revolute, parent link_2, child link_3, origin xyz=1.350 0 0, axis 0 1 0, limit lower=-2.0 upper=2.5 effort=9000 velocity=2.0
- added joint joint_4: type revolute, parent link_4, child tool, origin xyz=0 0 -0.089084, axis 0 0 1, limit lower=-6.10865 upper=6.10865 effort=800 velocity=6.0
- added joint joint_5: type revolute, parent link_3, child link_4, origin xyz=1.400 0 0, axis 0 1 0, limit lower=-6.3 upper=6.3 effort=1500 velocity=4.0
